File: Modules/ESP32-C3/ESP32-C3/ESP32-C3.kicad_sch (KiCad schematic)
At the start: 0 parts

Commit message: BMP388 updated.
Parts:
- added C1, C10, C2, C3, C4, C5, C6, C7, C8, C9: C_Small, symbol Device:C_Small
- added C11, C12: ~, symbol Device:C_Small
- added L1: L_Small, symbol Device:L_Small
- added R1, R2, R3, R4, R5, R6: R, symbol Device:R
- added U1: ESP32-C3, Package_DFN_QFN:QFN-32-1EP_5x5mm_P0.5mm_EP3.7x3.7mm, symbol MCU_Espressif:ESP32-C3
- added Y1: Crystal_GND24, symbol Device:Crystal_GND24
Connections:
- new net: C10.1, U1.29 (XTAL_N), Y1.3
- new net: R4.1, U1.22 (SPICLK)
- new net: C9.1, R1.1, Y1.1
- new net: C11.1, L1.1, U1.1 (LNA_IN)
- new net: C12.1, L1.2
- new net: R2.1, U1.19 (SPIHD)
- new net: R3.1, U1.20 (SPIWP)
- new net: R5.1, U1.23 (SPID)
- new net: R6.1, U1.24 (SPIQ)
- new net: R1.2, U1.30 (XTAL_P)
- new net +3.3V: C1.1, C2.1, C3.1, C4.1, C5.1, C6.1, C7.1, C8.1, U1.11 (VDD3P3_RTC), U1.17 (VDD3P3_CPU), U1.18 (VDD_SPI), U1.2 (VDD3P3), U1.3 (VDD3P3), U1.31 (VDDA), U1.32 (VDDA)
- new net GND: C1.2, C10.2, C11.2, C12.2, C2.2, C3.2, C4.2, C5.2, C6.2, C7.2, C8.2, C9.2, U1.33 (GND), Y1.2, Y1.4
- new net GPIO10: U1.16 (GPIO10)
- new net GPIO4: U1.9 (MTMS)
- new net GPIO5: U1.10 (MTDI)
- new net GPIO6: U1.12 (MTCK)
- new net GPIO7: U1.13 (MTDO)
- new net GPIO8: U1.14 (GPIO8)
- new net GPIO9: U1.15 (GPIO9)
- new net SPICLK: R4.2
- new net SPICS0: U1.21 (SPICS0)
- new net SPID: R5.2
- new net SPIHD: R2.2
- new net SPIQ: R6.2
- new net SPIWP: R3.2
