File: Modules/VOLTAGE_R/VOLTAGE_R.kicad_sch (KiCad schematic)
At the start: 7 parts, among them U1 TPS5430DDA

Commit message: ESP32-C3 Updated.
Parts:
- removed C1, C2, C3: C_Small, symbol Device:C_Small
- removed L1: L, symbol Device:L
- removed R1, R2: R_Small, symbol Device:R_Small
- removed U1: TPS5430DDA, Package_SO:TI_SO-PowerPAD-8_ThermalVias, symbol Regulator_Switching:TPS5430DDA
Connections:
- no-connect marks 1 -> 0

Commit message: Voltage Regulator updated
Parts:
- added C1: 430pF, symbol Device:C
- added C2: 10uF, symbol Device:C
- added C3: 47uF, symbol Device:C
- added PS1: TPS82140SILR, TPS82140SILR:CONV_TPS82140SILR, symbol TPS82140SILR:TPS82140SILR
- added R1: 10k, symbol Device:R
- added R2: 523k, symbol Device:R
- added R3: 100k, symbol Device:R
Connections:
- new net: PS1.7 (PG), R1.1
- new net: PS1.6 (FB), R2.1, R3.2
- new net: C1.1, PS1.8 (SS/TR)
- new net GND: C1.2, C2.1, C2.2, C3.1, C3.2, PS1.1 (EN), PS1.10 (GND), PS1.11 (GND), PS1.12 (GND), PS1.2 (VIN), PS1.3 (GND), PS1.4 (VOUT), PS1.5 (VOUT), PS1.9 (GND), R1.2, R2.2, R3.1
Other:
- note added: "YENIAY"
- title: (none) -> Voltage Regulator

Commit message: VoltageR updated
Parts:
- added C10: 22uF, symbol Device:C
- added C11: 68pF, symbol Device:C
- added C12, C8: 47uF, symbol Device:C
- added C4, C6, C9: 100uF, symbol Device:C
- added C5: 15uF, symbol Device:C
- added C7: 100pF, symbol Device:C
- added L1: 2.2uH, symbol Device:L
- added L2: 6.8uH, symbol Device:L
- added R4, R8: 100k, symbol Device:R
- added R5: 45.3k, symbol Device:R
- added R6: 10k, symbol Device:R
- added R7: 20k, symbol Device:R
- added R9: 13.7k, symbol Device:R
- added U1: TPS56637RPAR, TPS56637RPAR:CONV_TPS56637RPAR, symbol TPS56637RPAR:TPS56637RPAR
- added U2: TPS54202DDCR, TPS54202DDCR:SOT95P280X110-6N, symbol TPS54202DDCR:TPS54202DDCR
Connections:
- net GND: now also C10.1, C10.2, C11.1, C12.1, C12.2, C4.1, C4.2, C5.1, C5.2, C8.1, C8.2, L1.2, L2.2, R4.2, R5.2, R6.1, R7.2, R8.2, R9.1, U1.10 (MODE), U1.3 (AGND), U1.8 (VIN), U1.9 (PGND), U2.1 (GND), U2.3 (VIN)
- new net: C7.1, R5.1, R6.2, U1.2 (FB)
- new net: C9.1, U2.6 (BOOT)
- new net: C9.2, L2.1, U2.2 (SW)
- new net: C11.2, R8.1, R9.2, U2.4 (FB)
- new net: C7.2, R7.1
- new net: C6.1, U1.7 (BOOT)
- new net: C6.2, L1.1, U1.6 (SW)
- new net: R4.1, U1.4 (PG)
Other:
- note added: "TPS54202DDCR will be used"
- moved on the sheet: C1, C2, C3, PS1, R1, R2, R3

Commit message: EEPROM
Parts:
- added U3: 24AA64T-I/OT, SOT-23-5_MC_MCH, symbol 2024-04-16_22-30-30:24AA64T-I_OT
Connections:
- net GND: now also U3.2 (VSS), U3.5 (WP)
- new net +3.3V: U3.4 (VCC)
- new net I2C1_SCL: U3.1 (SCL)
- new net I2C1_SDA: U3.3 (SDA)
