File: CC_M7/ControlComputer.kicad_sch (KiCad schematic)
At the start: 38 parts, among them U1 STM32H743VITx, Y1 32MHz

Commit message: Routing Progress | BMM150 removed.
Other:
- note added: "KRISTAL KAPASITORLERI DEGISECEK"
Changed lines of the file:
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@@
+		)
+	)
+	(text "KRISTAL KAPASITORLERI DEGISECEK\n"
+		(exclude_from_sim no)
+		(at 226.06 104.14 0)
+		(effects
+			(font
+				(size 3.81 3.81)
+				(thickness 0.762)
+				(bold yes)
+			)
 		)
 	)

Commit message: USB Pullup added, oscillator capacitors updated.
Parts:
- C20, C21: value 12pF -> 16pF
Other:
- note removed: "KRISTAL KAPASITORLERI DEGISECEK"
- note removed: "USB D+ HATTINA 1.5 K ile PULLUP 3.3V EKLENECEK"
Changed lines of the file:
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@@
-		)
-	)
-	(text "KRISTAL KAPASITORLERI DEGISECEK\n"
-		(exclude_from_sim no)
-		(at 226.06 104.14 0)
-		(effects
-			(font
-				(size 3.81 3.81)
-				(thickness 0.762)
-				(bold yes)
-			)
 		)
 	)
@@
 				(bold yes)
 				(italic yes)
-			)
-		)
-	)
-	(text "USB D+ HATTINA 1.5 K ile PULLUP 3.3V EKLENECEK"
-		(exclude_from_sim no)
-		(at 70.485 133.985 0)
-		(effects
-			(font
-				(size 3.81 3.81)
-				(thickness 0.762)
-				(bold yes)
 			)
 		)
@@
 			)
 		)
-		(property "Value" "12pF"
+		(property "Value" "16pF"
 			(at 147.574 112.776 0)
 			(effects
@@
 			)
 		)
-		(property "Value" "12pF"
+		(property "Value" "16pF"
 			(at 171.45 111.7662 0)
 			(effects

Commit message: warning check
Parts:
- JP1, JP2, JP3, JP4: footprint Jumper:SolderJumper-2_P1.3mm_Open_TrianglePad1.0x1.5mm -> jmpertest:jmpertest
Changed lines of the file:
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@@
 			)
 		)
-		(property "Footprint" "Jumper:SolderJumper-2_P1.3mm_Open_TrianglePad1.0x1.5mm"
+		(property "Footprint" "jmpertest:jmpertest"
 			(at 163.83 219.71 0)
 			(effects
@@
 			)
 		)
-		(property "Footprint" "Jumper:SolderJumper-2_P1.3mm_Open_TrianglePad1.0x1.5mm"
+		(property "Footprint" "jmpertest:jmpertest"
 			(at 163.83 209.55 0)
 			(effects
@@
 			)
 		)
-		(property "Footprint" "Jumper:SolderJumper-2_P1.3mm_Open_TrianglePad1.0x1.5mm"
+		(property "Footprint" "jmpertest:jmpertest"
 			(at 163.83 214.63 0)
 			(effects
@@
 			)
 		)
-		(property "Footprint" "Jumper:SolderJumper-2_P1.3mm_Open_TrianglePad1.0x1.5mm"
+		(property "Footprint" "jmpertest:jmpertest"
 			(at 163.83 204.47 0)
 			(effects
