File: CC_M7/CC_M7.kicad_pcb (KiCad board)
At the start: 4 copper layers, 40 x 65 mm, 129 parts, among them J1 Conn_01x04_Pin, J10 Conn_01x04_Pin, J11 USB_B_Micro, J12 Conn_01x04_Pin, J13 Batt_Pins, J3 Conn_01x03_Pin, J4 Conn_01x03_Pin, J5 Conn_01x03_Pin, J6 Conn_01x03_Pin, J7 Conn_01x03_Pin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

Commit message: error chekc
Routing:
- net SPI1_CS3: track 5.57 -> 9.07 mm, vias 1 -> 2
- net DEC5: track 1.21 -> 2.33 mm
- net Net-(U8-FB): vias 2 -> 1
- net I2C1_SCL: vias 4 -> 5
- net GND: vias 16 -> 17
Changed lines of the file:
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@@
 		(attr through_hole)
 		(fp_line
-			(start -1.33 -1.33)
-			(end 0 -1.33)
-			(stroke
-				(width 0.12)
-				(type solid)
-			)
-			(layer "F.SilkS")
-		)
-		(fp_line
-			(start -1.33 0)
-			(end -1.33 -1.33)
-			(stroke
-				(width 0.12)
-				(type solid)
-			)
-			(layer "F.SilkS")
-		)
-		(fp_line
-			(start 1.33 1.27)
-			(end 1.33 6.41)
-			(stroke
-				(width 0.12)
-				(type solid)
-			)
-			(layer "F.SilkS")
-		)
-		(fp_line
-			(start -1.33 1.27)
-			(end 1.33 1.27)
-			(stroke
-				(width 0.12)
-				(type solid)
-			)
-			(layer "F.SilkS")
-		)
-		(fp_line
-			(start -1.33 1.27)
-			(end -1.33 6.41)
-			(stroke
-				(width 0.12)
-				(type solid)
-			)
-			(layer "F.SilkS")
-		)
-		(fp_line
-			(start -1.33 6.41)
-			(end 1.33 6.41)
-			(stroke
-				(width 0.12)
-				(type solid)
-			)
-			(layer "F.SilkS")
-		)
-		(fp_line
 			(start 1.8 -1.8)
 			(end -1.8 -1.8)
@@
 			(layer "F.CrtYd")
 		)
-		(fp_line
-			(start 1.27 -1.27)
-			(end 1.27 6.35)
-			(stroke
-				(width 0.1)
-				(type solid)
-			)
-			(layer "F.Fab")
-		)
-		(fp_line
-			(start -0.635 -1.27)
-			(end 1.27 -1.27)
-			(stroke
-				(width 0.1)
-				(type solid)
-			)
-			(layer "F.Fab")
-		)
-		(fp_line
-			(start -1.27 -0.635)
-			(end -0.635 -1.27)
-			(stroke
-				(width 0.1)
-				(type solid)
-			)
-			(layer "F.Fab")
-		)
-		(fp_line
-			(start 1.27 6.35)
-			(end -1.27 6.35)
-			(stroke
-				(width 0.1)
-				(type solid)
-			)
-			(layer "F.Fab")
-		)
-		(fp_line
-			(start -1.27 6.35)
-			(end -1.27 -0.635)
-			(stroke
-				(width 0.1)
-				(type solid)
-			)
-			(layer "F.Fab")
-		)
 		(fp_text user "${REFERENCE}"
 			(at 0 2.54 0)
@@
 		)
 	)
-	(gr_text "+   -"
-		(at 124.72 167.16 -90)
+	(gr_text "+  -"
+		(at 124.72 167.16 270)
 		(layer "B.SilkS" knockout)
 		(effects
 			(font
-				(face "Artifakt Element Black")
-				(size 2.2 2.2)
+				(face "Pointless")
+				(size 1.4 1.4)
 				(thickness 0.125)
 				(bold yes)
@@
 			(justify left bottom mirror)
 		)
-		(render_cache "+   -" 270
+		(render_cache "+  -" 270
 			(polygon
 				(pts
-					(xy 125.953734 165.62591) (xy 125.953734 166.023538) (xy 125.541062 166.023538) (xy 125.541062 166.457704)
-					(xy 125.953734 166.457704) (xy 125.953734 166.855331) (xy 126.366407 166.855331) (xy 126.366407 166.457704)
-					(xy 126.77908 166.457704) (xy 126.77908 166.023538) (xy 126.366407 166.023538) (xy 126.366407 165.62591)
+					(xy 124.958 166.424487) (xy 125.691119 166.424487) (xy 125.691119 167.16) (xy 126.205397 167.16)
+					(xy 126.205397 166.424487) (xy 126.949458 166.424487) (xy 126.949458 165.912602) (xy 126.205397 165.912602)
+					(xy 126.205397 165.168541) (xy 125.691119 165.168541) (xy 125.691119 165.912602) (xy 124.958 165.912602)
 				)
 			)
 			(polygon
 				(pts
-					(xy 125.953734 161.927438) (xy 125.953734 162.928492) (xy 126.366407 162.928492) (xy 126.366407 161.927438)
+					(xy 125.702061 163.047145) (xy 126.216339 163.047145) (xy 126.216339 161.559023) (xy 125.702061 161.559023)
 				)
 			)
@@
 		)
 	)
-	(gr_text "+   -"
-		(at 127.62 167.16 90)
-		(layer "F.SilkS" knockout)
-		(effects
-			(font
-				(face "Artifakt Element Black")
-				(size 2.2 2.2)
-				(thickness 0.125)
-				(bold yes)
-			)
-			(justify left bottom)
-		)
-		(render_cache "+   -" 90
-			(polygon
-				(pts
-					(xy 126.386265 165.62591) (xy 126.386265 166.023538) (xy 126.798937 166.023538) (xy 126.798937 166.457704)
-					(xy 126.386265 166.457704) (xy 126.386265 166.855331) (xy 125.973592 166.855331) (xy 125.973592 166.457704)
-					(xy 125.560919 166.457704) (xy 125.560919 166.023538) (xy 125.973592 166.023538) (xy 125.973592 165.62591)
-				)
-			)
-			(polygon
-				(pts
-					(xy 126.386265 161.927438) (xy 126.386265 162.928492) (xy 125.973592 162.928492) (xy 125.973592 161.927438)
-				)
-			)
-		)
-	)
 	(gr_text "BTX"
 		(at 113.05 155.45 0)
@@
 	)
 	(via
+		(at 111.78 142.42)
+		(size 0.35)
+		(drill 0.2)
+		(layers "F.Cu" "B.Cu")
+		(free yes)
+		(net 1)
+	)
+	(via
 		(at 102.7 154.3)
 		(size 0.35)
@@
 	)
 	(segment
+		(start 109.275 118.1292)
+		(end 109.275 119.148367)
+		(width 0.2)
+		(layer "B.Cu")
+		(net 17)
+	)
+	(segment
+		(start 109.275 119.148367)
+		(end 109.205067 119.2183)
+		(width 0.2)
+		(layer "B.Cu")
+		(net 17)
+	)
+	(segment
 		(start 106.95 118.4)
 		(end 106.930837 118.4)
@@
 	)
 	(segment
-		(start 102.6517 122.5653)
-		(end 102.5906 122.5042)
-		(width 0.15)
-		(layer "F.Cu")
-		(net 18)
-	)
-	(segment
 		(start 101.86 122.135)
 		(end 102.2292 122.5042)
@@
 	)
 	(segment
-		(start 97.8162 158.1912)
-		(end 97.8 158.175)
-		(width 0.5)
-		(layer "In2.Cu")
-		(net 19)
-	)
-	(segment
 		(start 99.8728 123.149834)
 		(end 99.8728 123.1392)
@@
 		(net 24)
 	)
-	(via
-		(at 110.8202 161.542)
-		(size 0.6)
-		(drill 0.3)
-		(layers "F.Cu" "B.Cu")
-		(net 24)
-	)
 	(segment
 		(start 112.395 161.543)
@@
 	(segment
 		(start 104.625 156.525)
+		(end 104.605 156.545)
+		(width 0.2)
+		(layer "F.Cu")
+		(net 35)
+	)
+	(segment
+		(start 104.605 156.545)
 		(end 104.6 156.55)
 		(width 0.2)
@@
 	)
 	(via
+		(at 104.599997 156.550003)
+		(size 0.35)
+		(drill 0.2)
+		(layers "F.Cu" "B.Cu")
+		(net 35)
+	)
+	(via
 		(at 97.15 127.8)
 		(size 0.35)
@@
 	)
 	(segment
-		(start 95 151.6)
-		(end 95 151.5)
-		(width 0.2)
-		(layer "In1.Cu")
-		(net 46)
-	)
-	(segment
 		(start 103.754578 147.674843)
 		(end 103.745421 147.684)
@@
 	)
 	(segment
-		(start 109.992554 119.25)
-		(end 109.992559 119.250005)
-		(width 0.15)
-		(layer "In2.Cu")
-		(net 84)
-	)
-	(segment
 		(start 102.365686 118.3)
 		(end 103.11 119.044314)
@@
 	)
 	(segment
+		(start 105.267 143.253)
+		(end 105.5 143.02)
+		(width 0.2)
+		(layer "F.Cu")
+		(net 121)
+	)
+	(segment
+		(start 105.267 144.382)
+		(end 105.267 143.253)
+		(width 0.2)
+		(layer "F.Cu")
+		(net 121)
+	)
+	(segment
 		(start 108.6785 146.66)
 		(end 108.6785 146.6)
@@
 		(net 121)
 	)
+	(via
+		(at 105.5 143.02)
+		(size 0.35)
+		(drill 0.2)
+		(layers "F.Cu" "B.Cu")
+		(net 121)
+	)
 	(segment
-		(start 105.2758 145.25)
-		(end 107.975 145.25)
+		(start 105.5 143.03)
+		(end 105.5 143.02)
+		(width 0.2)
+		(layer "In2.Cu")
+		(net 121)
+	)
+	(segment
+		(start 105.27 144.75)
+		(end 105.27 143.26)
+		(width 0.2)
+		(layer "In2.Cu")
+		(net 121)
+	)
+	(segment
+		(start 105.77 145.25)
+		(end 105.27 144.75)
+		(width 0.2)
+		(layer "In2.Cu")
+		(net 121)
+	)
+	(segment
+		(start 108.6785 146.6)
+		(end 108.6785 145.9535)
+		(width 0.2)
+		(layer "In2.Cu")
+		(net 121)
+	)
+	(segment
+		(start 105.27 143.26)
+		(end 105.5 143.03)
 		(width 0.2)
 		(layer "In2.Cu")
@@
 	(segment
 		(start 108.6785 145.9535)
-		(end 108.6785 146.6)
+		(end 107.975 145.25)
 		(width 0.2)
 		(layer "In2.Cu")
@@
 	(segment
 		(start 107.975 145.25)
-		(end 108.6785 145.9535)
+		(end 105.77 145.25)
 		(width 0.2)
 		(layer "In2.Cu")

Commit message: Error check
Routing:
- net +3.3V: track 48.5 -> 66.1 mm, vias 13 -> 16
- net GND: track 51.8 -> 67.3 mm, vias 17 -> 25
- net NRST: track 49.2 -> 55.1 mm, vias 3 -> 4
- net USB_DP: track 57.6 -> 59.0 mm
- net Net-(C18-Pad1): track 5.81 -> 7.09 mm
- net I2C1_SCL: vias 5 -> 6
