File: CC_M7/Sensors.kicad_sch (KiCad schematic)
At the start: 18 parts, among them U11 BMP581, U12 IIM-42652, U2 24AA64T-I/OT, U3 BMI088, U4 ICP-20100, U5 BMM150

Commit message: BOM added.
Parts:
- C51: value C_Small -> 100nF
- C52: value C_Small -> 2.2uF
- C53: value C_Small -> 10nF
Changed lines of the file:
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@@
 			)
 		)
-		(property "Value" "C_Small"
+		(property "Value" "100nF"
 			(at 144.78 26.6762 0)
 			(effects
@@
 			)
 		)
-		(property "Value" "C_Small"
+		(property "Value" "2.2uF"
 			(at 157.48 26.6762 0)
 			(effects
@@
 			)
 		)
-		(property "Value" "C_Small"
+		(property "Value" "10nF"
 			(at 170.18 26.6762 0)
 			(effects
